File: hardware/ultra-violet-tooth-sensor-mk-3.3.brd (EAGLE design)
At the start: 39 x 28 mm, 20 parts, among them Q1 IRLML2244, U1 RFDUINOSMD, U2 ADAFRUIT-SI1145-BREAKOUTNOHOL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

Commit message: more dicking around
Parts:
- removed BAT1: CR2032, A_butts:BATTCON_20MM_MINE_STAHPIT
- added U3: MCP73831, A_butts:SOT95P280X145-5N
- moved TX 21.8 mm to (11.0, 15.2), turned to 0 degrees
- moved RX 15.5 mm to (11.0, 12.8)
- moved JP1 13.2 mm to (42.0, 16.0)
- moved C1 12.0 mm to (18.0, 17.0), flipped to the top
- moved Q1 9.12 mm to (18.1, 22.0), flipped to the top
- moved GPIO4 9.01 mm to (7.00, 26.0), turned to 180 degrees
- moved GPIO3 7.02 mm to (12.0, 26.0), turned to 180 degrees
- moved POWER 5.80 mm to (27.0, 26.0)
- moved BATT 5.50 mm to (18.0, 26.0), flipped to the bottom
- moved U2 1.00 mm to (29.0, 14.0), turned to 270 degrees
- moved R2 0.25 mm to (12.0, 25.5), flipped to the bottom, turned to 180 degrees
- moved R3 0.25 mm to (6.75, 25.5), flipped to the bottom, turned to 180 degrees
- moved U$2 0.25 mm to (4.75, 14.0)
Connections:
- new net N$3: U3.4
- new net VBATT: BATT.2, POWER.3
- new net VSS: U3.2
- net GND: no longer BAT1.BOTTOM
- net N$1: now also U3.3; no longer BAT1.TOP@1, BATT.2, POWER.3
Routing:
- net VCC: track 66.7 -> 7.37 mm, vias 2 -> 0
- net SCL: track 31.5 -> 4.39 mm, vias 0 -> 1
- net GPIO0: track 25.0 -> 0.00 mm, vias 1 -> 0
- net SDA: track 29.6 -> 6.02 mm, vias 0 -> 1
- net GPIO1: track 20.3 -> 0.00 mm, vias 1 -> 0
- net INT_SI1145: track 17.6 -> 0.00 mm
- net N$1: track 15.7 -> 0.00 mm
- net RXD: track 11.1 -> 0.00 mm, vias 1 -> 0
- net DFU: track 9.85 -> 0.00 mm, vias 1 -> 0
- net RST: track 6.79 -> 0.00 mm
- net GPIO3: track 11.8 -> 5.10 mm
- net N$2: track 5.50 -> 0.00 mm
- net TXD: track 4.99 -> 0.00 mm, vias 1 -> 0
- net GPIO4: track 9.57 -> 5.44 mm
Other:
- board text added: "GPIO0"
- board text added: "GPIO1"
- board text removed: "0"
- board text removed: "1"

Commit message: more tweaking/twaddling
Parts:
- added D1: 10V, A_butts:SOT23
- added R1: 100k, A_butts:R0805
- JP1: value FTDI_CONNSMT -> FTDI_CONNJST-PH-SMD-RA; device A_butts:FTDI_CONN_SMT -> A_butts:AVRISP-JST-6-PH-RA-SMD
- Q1: value IRLML2244 -> IRLML2502; device A_butts:SOT23-3 -> A_butts:SOT23
- moved JP1 19.6 mm to (24.0, 8.25), turned to 180 degrees
- moved C1 11.0 mm to (17.0, 6.00)
- moved U3 3.01 mm to (15.0, 21.0)
- moved Q1 1.38 mm to (19.0, 21.0), flipped to the bottom
- moved U2 1.25 mm to (27.8, 14.0), turned to 90 degrees
- moved RX 0.25 mm to (11.2, 12.8)
- moved TX 0.25 mm to (11.2, 15.2)
Connections:
- net VBATT renamed BATT+
- removed net N$2: POWER.2, Q1.3
- new net BATT-: BATT.1, Q1.3
- new net N$4: D1.3, Q1.1, R1.1
- net GND: now also D1.1, D1.2, Q1.2; no longer BATT.1, Q1.1
- net VCC: now also POWER.2, R1.2; no longer Q1.2
