File: hardware/ultra-violet-tooth-sensor-mk-3.3.sch (EAGLE design)
At the start: 17 parts, among them Q1 IRLML2244, U1 RFDUINOSMD, U2 ADAFRUIT-SI1145-BREAKOUTNOHOL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

Commit message: more dicking around
Parts:
- removed BAT1: CR2032, A_butts:BATTERY-COINCR2032_SMD_TIGHT
- added U3: MCP73831, A_butts:MCP73831T-2ACI/OT
Connections:
- new net N$3: U3.VDD
- new net VBATT: BATT.2, POWER.NO
- net GND: no longer BAT1.-
- net N$1: now also U3.VBAT; no longer BAT1.+, BATT.2, POWER.NO
Changed lines of the file:
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@@
 <part name="SUPPLY5" library="A_butts" deviceset="VCC" device=""/>
 <part name="GND2" library="A_butts" deviceset="GND" device=""/>
-<part name="BAT1" library="A_butts" deviceset="BATTERY-COIN" device="CR2032_SMD_TIGHT" value="CR2032"/>
 <part name="R2" library="A_butts" deviceset="RESISTOR" device="R0805" value="10k"/>
 <part name="R3" library="A_butts" deviceset="RESISTOR" device="R0805" value="10k"/>
@@
 <part name="DFU" library="A_butts" deviceset="M01" device="SMD_1.5X2MM" value="M01SMD_1.5X2MM"/>
 <part name="JP1" library="A_butts" deviceset="FTDI_CONN" device="SMT" value="FTDI_CONNSMT"/>
+<part name="U3" library="A_butts" deviceset="MCP73831T-2ACI/OT" device="" value="MCP73831"/>
 </parts>
 <sheets>
@@
 <instance part="POWER" gate="G$1" x="167.64" y="116.84"/>
 <instance part="SUPPLY6" gate="G$1" x="160.02" y="139.7"/>
-<instance part="GND6" gate="1" x="185.42" y="93.98"/>
+<instance part="GND6" gate="1" x="185.42" y="106.68"/>
 <instance part="BATT" gate="G$1" x="198.12" y="109.22" rot="MR0"/>
 <instance part="U1" gate="G$1" x="38.1" y="109.22"/>
@@
 <instance part="SUPPLY5" gate="G$1" x="25.4" y="78.74"/>
 <instance part="GND2" gate="1" x="25.4" y="60.96"/>
-<instance part="BAT1" gate="G$1" x="175.26" y="106.68" rot="R270"/>
 <instance part="R2" gate="G$1" x="111.76" y="139.7"/>
 <instance part="R3" gate="G$1" x="111.76" y="132.08"/>
@@
 <instance part="DFU" gate="G$1" x="99.06" y="88.9" rot="MR0"/>
 <instance part="JP1" gate="G$1" x="86.36" y="160.02"/>
+<instance part="U3" gate="A" x="167.64" y="73.66"/>
 </instances>
 <busses>
@@
 <segment>
 <pinref part="GND6" gate="1" pin="GND"/>
-<wire x1="185.42" y1="96.52" x2="185.42" y2="99.06" width="0.1524" layer="91"/>
-<wire x1="185.42" y1="99.06" x2="185.42" y2="111.76" width="0.1524" layer="91"/>
+<wire x1="185.42" y1="109.22" x2="185.42" y2="111.76" width="0.1524" layer="91"/>
 <wire x1="185.42" y1="111.76" x2="187.96" y2="111.76" width="0.1524" layer="91"/>
 <pinref part="BATT" gate="G$1" pin="1"/>
-<pinref part="BAT1" gate="G$1" pin="-"/>
-<wire x1="175.26" y1="101.6" x2="175.26" y2="99.06" width="0.1524" layer="91"/>
-<wire x1="175.26" y1="99.06" x2="185.42" y2="99.06" width="0.1524" layer="91"/>
-<junction x="185.42" y="99.06"/>
+<junction x="185.42" y="111.76"/>
 <pinref part="Q1" gate="G$1" pin="G"/>
 <wire x1="152.4" y1="129.54" x2="149.86" y2="129.54" width="0.1524" layer="91"/>
-<wire x1="149.86" y1="129.54" x2="149.86" y2="99.06" width="0.1524" layer="91"/>
-<wire x1="149.86" y1="99.06" x2="175.26" y2="99.06" width="0.1524" layer="91"/>
-<junction x="175.26" y="99.06"/>
+<wire x1="149.86" y1="129.54" x2="149.86" y2="111.76" width="0.1524" layer="91"/>
+<wire x1="149.86" y1="111.76" x2="185.42" y2="111.76" width="0.1524" layer="91"/>
 </segment>
 <segment>
@@
 </segment>
 </net>
-<net name="N$1" class="0">
+<net name="VBATT" class="0">
 <segment>
 <pinref part="BATT" gate="G$1" pin="2"/>
-<pinref part="BAT1" gate="G$1" pin="+"/>
-<wire x1="175.26" y1="114.3" x2="187.96" y2="114.3" width="0.1524" layer="91"/>
-<wire x1="175.26" y1="114.3" x2="175.26" y2="111.76" width="0.1524" layer="91"/>
+<wire x1="172.72" y1="114.3" x2="187.96" y2="114.3" width="0.1524" layer="91"/>
 <pinref part="POWER" gate="G$1" pin="NO"/>
-<wire x1="172.72" y1="114.3" x2="175.26" y2="114.3" width="0.1524" layer="91"/>
-<junction x="175.26" y="114.3"/>
+<label x="180.34" y="116.84" size="1.27" layer="95"/>
 </segment>
 </net>
@@
 </segment>
 </net>
+<net name="N$1" class="0">
+<segment>
+<pinref part="U3" gate="A" pin="VBAT"/>
+<wire x1="187.96" y1="78.74" x2="185.42" y2="78.74" width="0.1524" layer="91"/>
+</segment>
+</net>
+<net name="N$3" class="0">
+<segment>
+<wire x1="147.32" y1="81.28" x2="147.32" y2="78.74" width="0.1524" layer="91"/>
+<pinref part="U3" gate="A" pin="VDD"/>
+<wire x1="147.32" y1="78.74" x2="149.86" y2="78.74" width="0.1524" layer="91"/>
+</segment>
+</net>

Commit message: more tweaking/twaddling
Parts:
- added D1: 10V, A_butts:DIODE-ZENERSOT23
- added R1: 100k, A_butts:RESISTORR0805
- JP1: value FTDI_CONNSMT -> FTDI_CONNJST-PH-SMD-RA; device A_butts:FTDI_CONNSMT -> A_butts:FTDI_CONNJST-PH-SMD-RA
- Q1: value IRLML2244 -> IRLML2502; device A_butts:MOSFET-PCHANNELIRLML2244 -> A_butts:MOSFET-NCHANNELIRLML2502
Connections:
- net VBATT renamed BATT+
- removed net N$2: POWER.COM, Q1.D
- new net BATT-: BATT.1, Q1.D
- new net N$4: D1.C, Q1.G, R1.1
- net GND: now also D1.A, Q1.S; no longer BATT.1, Q1.G
- net VCC: now also POWER.COM, R1.2; no longer Q1.S
Other:
- moved on the sheet: Q1, U3
Changed lines of the file:
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@@
 <part name="R3" library="A_butts" deviceset="RESISTOR" device="R0805" value="10k"/>
 <part name="SUPPLY4" library="A_butts" deviceset="VCC" device=""/>
-<part name="Q1" library="A_butts" deviceset="MOSFET-PCHANNEL" device="IRLML2244" value="IRLML2244"/>
 <part name="C1" library="A_butts" deviceset="CAPACITOR-CERAMIC" device="C1206" value="10uF"/>
 <part name="SUPPLY2" library="A_butts" deviceset="VCC" device=""/>
@@
 <part name="GPIO4" library="A_butts" deviceset="M01" device="SMD_1.5X2MM" value="M01SMD_1.5X2MM"/>
 <part name="DFU" library="A_butts" deviceset="M01" device="SMD_1.5X2MM" value="M01SMD_1.5X2MM"/>
-<part name="JP1" library="A_butts" deviceset="FTDI_CONN" device="SMT" value="FTDI_CONNSMT"/>
+<part name="JP1" library="A_butts" deviceset="FTDI_CONN" device="JST-PH-SMD-RA" value="FTDI_CONNJST-PH-SMD-RA"/>
 <part name="U3" library="A_butts" deviceset="MCP73831T-2ACI/OT" device="" value="MCP73831"/>
+<part name="Q1" library="A_butts" deviceset="MOSFET-NCHANNEL" device="IRLML2502" value="IRLML2502"/>
+<part name="R1" library="A_butts" deviceset="RESISTOR" device="R0805" value="100k"/>
+<part name="D1" library="A_butts" deviceset="DIODE-ZENER" device="SOT23" value="10V"/>
 </parts>
 <sheets>
@@
 <instance part="SUPPLY3" gate="G$1" x="20.32" y="119.38"/>
 <instance part="POWER" gate="G$1" x="167.64" y="116.84"/>
-<instance part="SUPPLY6" gate="G$1" x="160.02" y="139.7"/>
-<instance part="GND6" gate="1" x="185.42" y="106.68"/>
+<instance part="SUPPLY6" gate="G$1" x="160.02" y="124.46"/>
+<instance part="GND6" gate="1" x="172.72" y="86.36"/>
 <instance part="BATT" gate="G$1" x="198.12" y="109.22" rot="MR0"/>
 <instance part="U1" gate="G$1" x="38.1" y="109.22"/>
@@
 <instance part="R3" gate="G$1" x="111.76" y="132.08"/>
 <instance part="SUPPLY4" gate="G$1" x="119.38" y="142.24"/>
-<instance part="Q1" gate="G$1" x="160.02" y="129.54" rot="MR180"/>
 <instance part="C1" gate="G$1" x="190.5" y="162.56"/>
 <instance part="SUPPLY2" gate="G$1" x="190.5" y="170.18"/>
@@
 <instance part="DFU" gate="G$1" x="99.06" y="88.9" rot="MR0"/>
 <instance part="JP1" gate="G$1" x="86.36" y="160.02"/>
-<instance part="U3" gate="A" x="167.64" y="73.66"/>
+<instance part="U3" gate="A" x="170.18" y="50.8"/>
+<instance part="Q1" gate="G$1" x="172.72" y="101.6"/>
+<instance part="R1" gate="G$1" x="160.02" y="109.22" rot="R90"/>
+<instance part="D1" gate="G$1" x="160.02" y="96.52" rot="R90"/>
 </instances>
 <busses>
@@
 <wire x1="20.32" y1="116.84" x2="22.86" y2="116.84" width="0.1524" layer="91"/>
 <pinref part="U1" gate="G$1" pin="3V"/>
-</segment>
-<segment>
-<pinref part="SUPPLY6" gate="G$1" pin="VCC"/>
-<pinref part="Q1" gate="G$1" pin="S"/>
-<wire x1="160.02" y1="139.7" x2="160.02" y2="134.62" width="0.1524" layer="91"/>
 </segment>
 <segment>
@@
 <wire x1="190.5" y1="170.18" x2="190.5" y2="167.64" width="0.1524" layer="91"/>
 </segment>
+<segment>
+<wire x1="160.02" y1="124.46" x2="160.02" y2="116.84" width="0.1524" layer="91"/>
+<pinref part="POWER" gate="G$1" pin="COM"/>
+<wire x1="160.02" y1="116.84" x2="162.56" y2="116.84" width="0.1524" layer="91"/>
+<pinref part="SUPPLY6" gate="G$1" pin="VCC"/>
+<pinref part="R1" gate="G$1" pin="2"/>
+<wire x1="160.02" y1="114.3" x2="160.02" y2="116.84" width="0.1524" layer="91"/>
+<junction x="160.02" y="116.84"/>
+</segment>
 </net>
 <net name="GND" class="0">
@@
 <pinref part="GND1" gate="1" pin="GND"/>
 <wire x1="200.66" y1="157.48" x2="200.66" y2="154.94" width="0.1524" layer="91"/>
-</segment>
-<segment>
-<pinref part="GND6" gate="1" pin="GND"/>
-<wire x1="185.42" y1="109.22" x2="185.42" y2="111.76" width="0.1524" layer="91"/>
-<wire x1="185.42" y1="111.76" x2="187.96" y2="111.76" width="0.1524" layer="91"/>
-<pinref part="BATT" gate="G$1" pin="1"/>
-<junction x="185.42" y="111.76"/>
-<pinref part="Q1" gate="G$1" pin="G"/>
-<wire x1="152.4" y1="129.54" x2="149.86" y2="129.54" width="0.1524" layer="91"/>
-<wire x1="149.86" y1="129.54" x2="149.86" y2="111.76" width="0.1524" layer="91"/>
-<wire x1="149.86" y1="111.76" x2="185.42" y2="111.76" width="0.1524" layer="91"/>
 </segment>
 <segment>
@@
 <wire x1="190.5" y1="154.94" x2="190.5" y2="157.48" width="0.1524" layer="91"/>
 </segment>
+<segment>
+<pinref part="Q1" gate="G$1" pin="S"/>
+<pinref part="GND6" gate="1" pin="GND"/>
+<wire x1="172.72" y1="88.9" x2="172.72" y2="91.44" width="0.1524" layer="91"/>
+<pinref part="D1" gate="G$1" pin="A"/>
+<wire x1="172.72" y1="91.44" x2="172.72" y2="96.52" width="0.1524" layer="91"/>
+<wire x1="160.02" y1="93.98" x2="160.02" y2="91.44" width="0.1524" layer="91"/>
+<wire x1="160.02" y1="91.44" x2="172.72" y2="91.44" width="0.1524" layer="91"/>
+<junction x="172.72" y="91.44"/>
+</segment>
 </net>
 <net name="RST" class="0">
@@
 </segment>
 </net>
-<net name="VBATT" class="0">
+<net name="BATT+" class="0">
 <segment>
 <pinref part="BATT" gate="G$1" pin="2"/>
@@
 </segment>
 </net>
-<net name="N$2" class="0">
-<segment>
-<pinref part="Q1" gate="G$1" pin="D"/>
-<wire x1="160.02" y1="124.46" x2="160.02" y2="116.84" width="0.1524" layer="91"/>
-<pinref part="POWER" gate="G$1" pin="COM"/>
-<wire x1="160.02" y1="116.84" x2="162.56" y2="116.84" width="0.1524" layer="91"/>
-</segment>
-</net>
 <net name="INT_SI1145" class="0">
 <segment>
@@
 <segment>
 <pinref part="U3" gate="A" pin="VBAT"/>
-<wire x1="187.96" y1="78.74" x2="185.42" y2="78.74" width="0.1524" layer="91"/>
+<wire x1="190.5" y1="55.88" x2="187.96" y2="55.88" width="0.1524" layer="91"/>
 </segment>
 </net>
 <net name="N$3" class="0">
 <segment>
-<wire x1="147.32" y1="81.28" x2="147.32" y2="78.74" width="0.1524" layer="91"/>
+<wire x1="149.86" y1="58.42" x2="149.86" y2="55.88" width="0.1524" layer="91"/>
 <pinref part="U3" gate="A" pin="VDD"/>
-<wire x1="147.32" y1="78.74" x2="149.86" y2="78.74" width="0.1524" layer="91"/>
-</segment>
-</net>
+<wire x1="149.86" y1="55.88" x2="152.4" y2="55.88" width="0.1524" layer="91"/>
+</segment>
+</net>
+<net name="BATT-" class="0">
+<segment>
+<pinref part="Q1" gate="G$1" pin="D"/>
+<wire x1="172.72" y1="106.68" x2="172.72" y2="111.76" width="0.1524" layer="91"/>
+<pinref part="BATT" gate="G$1" pin="1"/>
+<wire x1="172.72" y1="111.76" x2="187.96" y2="111.76" width="0.1524" layer="91"/>
+<label x="180.34" y="109.22" size="1.27" layer="95"/>
+</segment>
+</net>
+<net name="N$4" class="0">
+<segment>
+<pinref part="R1" gate="G$1" pin="1"/>
+<pinref part="D1" gate="G$1" pin="C"/>
+<wire x1="160.02" y1="104.14" x2="160.02" y2="101.6" width="0.1524" layer="91"/>
+<pinref part="Q1" gate="G$1" pin="G"/>
+<wire x1="160.02" y1="101.6" x2="160.02" y2="99.06" width="0.1524" layer="91"/>
+<wire x1="160.02" y1="101.6" x2="165.1" y2="101.6" width="0.1524" layer="91"/>
+<junction x="160.02" y="101.6"/>
+</segment>
+</net>
